File: Display_Board_B/Display_Board.sch (KiCad schematic (older format))
At the start: 0 parts

Commit message: Add Creative Commons License  CC BY-SA 4.0
Other:
- note added: "This work is licensed under the Creative Commons Attribution-ShareAlike 4.0 International License.\nTo view a copy of this license, visit http://creativecommons.org/licenses/by-sa/4.0/\nor send a letter to Creative Commons, PO Box 1866, Mountain View, CA 94042, USA."
Changed lines of the file:
@@
-EESchema Schematic File Version 2  date 8/1/2015 10:16:52 AM
+EESchema Schematic File Version 2  date 8/2/2015 6:47:50 AM
 LIBS:power
 LIBS:device
@@
 Sheet 1 2
 Title "ODR-1 DISPLAY BOARD"
-Date "31 jul 2015"
+Date "2 aug 2015"
 Rev "B"
 Comp ""
@@
 Text Notes 5200 4950 0    50   ~ 0
 JUL 2015
+Text Notes 1200 7650 0    60   ~ 0
+This work is licensed under the Creative Commons Attribution-ShareAlike 4.0 International License.\nTo view a copy of this license, visit http://creativecommons.org/licenses/by-sa/4.0/\nor send a letter to Creative Commons, PO Box 1866, Mountain View, CA 94042, USA.
 $EndSCHEMATC
