File: OSC_Mixer_Board_A1/OSC_Mixer_Board.kicad_pcb (KiCad board)
At the start: 4 copper layers, 144.8 x 99.9 mm, 526 parts, among them J1 FM-10, J2 FM-12, J3 FM-12, J4 FM-12, J5 FM-12, J6 FM-12, J7 FM-12, J8 PJ-057AH, Q1 IRLML2060TRPBF, Q2 DMP4015SSSQ, Q3 BFU520A, T1 ETC1-1T-2TR, U1 L78M05AB, U10 STLM20W87F, U11 SI5351A, U12 NC7SZ74, U13 NC7SZ74, U14 FST3257, U15 FST3257, U16 TLV2462CD, U17 TLV2462CD, U18 FST3257, U19 LT6231, U2 FST3253, U20 LT6231, U3 FST3253, U4 FST3253, U5 FST3253, U6 NCP700BSN18, U7 FST3253, U8 FST3253, U9 NCP700BSN33, X1 25 MHz

Commit message: Add Creative Commons License  CC BY-SA 4.0
Parts:
- added G***: OSHW-logo_silkscreen-front_5mm, OSHW-logo_silkscreen-front_5mm, F.Cu at (100.7, 143.9)
Other:
- board text added: "This work is licensed under the Creative Commons Attribution-ShareAlike 4.0 International License. To view a copy of this license, visit http://creativecommons.org/licenses/by-sa/4.0/ or send a letter to Creative Commons, PO Box 1866, Mountain View, CA 94042, USA."
